File: esp8266/esp8266 breakout.sch (KiCad schematic (older format))
At the start: 12 parts, among them IC1 DS18B20, P1 power, P2 prog, P3 ftdi, P4 dust, U1 esp8266, U2 AP1117D33

Commit message: all libs inside project
Parts:
- removed P2: prog, Pin_Headers:Pin_Header_Straight_1x02, symbol CONN_01X02
- added SW1: SW_PUSH, Buttons_Switches_ThroughHole:SW_PUSH_SMALL, symbol SW_PUSH
- IC1: footprint Housings_TO-92:TO-92_Molded_Narrow -> onewire:1wire-TO92-
- U1: footprint kicadlibs:esp8266 -> custom:esp8266
Connections:
- wire segments 29 -> 28
Changed lines of the file:
@@
 EESchema Schematic File Version 2
-LIBS:esp8266 breakout-rescue
 LIBS:power
 LIBS:device
@@
 F 0 "U1" H 4750 4800 60  0000 C CNN
 F 1 "esp8266" H 5100 4800 60  0000 C CNN
-F 2 "kicadlibs:esp8266" H 5100 4550 60  0001 C CNN
+F 2 "custom:esp8266" H 5100 4550 60  0001 C CNN
 F 3 "" H 5100 4550 60  0000 C CNN
 	1    4450 4850
@@
 Wire Wire Line
 	3200 5350 3300 5350
-$Comp
-L CONN_01X02 P2
-U 1 1 55A12BD5
-P 3950 4200
-F 0 "P2" H 3950 4350 50  0000 C CNN
-F 1 "prog" V 4050 4200 50  0000 C CNN
-F 2 "Pin_Headers:Pin_Header_Straight_1x02" H 3950 4200 60  0001 C CNN
-F 3 "" H 3950 4200 60  0000 C CNN
-	1    3950 4200
-	1    0    0    -1
-$EndComp
-Wire Wire Line
-	3750 4250 3150 4250
-Wire Wire Line
-	3150 4150 3750 4150
-Text Label 3350 4250 0    60   ~ 0
+Wire Wire Line
+	3150 3900 2800 3900
+Text Label 2900 3900 0    60   ~ 0
 gpio0
 Wire Wire Line
@@
 Text Label 4100 5750 0    60   ~ 0
 tx
-Connection ~ 3350 4150
 $Comp
 L AP1117D33 U2
@@
 L GND #PWR011
 U 1 1 55A13B66
-P 3150 4150
-F 0 "#PWR011" H 3150 3900 50  0001 C CNN
-F 1 "GND" H 3150 4000 50  0000 C CNN
-F 2 "" H 3150 4150 60  0000 C CNN
-F 3 "" H 3150 4150 60  0000 C CNN
-	1    3150 4150
-	0    1    1    0
+P 3750 3900
+F 0 "#PWR011" H 3750 3650 50  0001 C CNN
+F 1 "GND" H 3750 3750 50  0000 C CNN
+F 2 "" H 3750 3900 60  0000 C CNN
+F 3 "" H 3750 3900 60  0000 C CNN
+	1    3750 3900
+	0    -1   -1   0
 $EndComp
 $Comp
@@
 F 0 "IC1" H 7125 4325 50  0000 L BNN
 F 1 "DS18B20" H 7125 4225 50  0000 L BNN
-F 2 "Housings_TO-92:TO-92_Molded_Narrow" H 6900 4450 50  0001 C CNN
+F 2 "onewire:1wire-TO92-" H 6900 4450 50  0001 C CNN
 F 3 "" H 6900 4300 60  0000 C CNN
 	2    6900 4300
@@
 F 0 "IC1" H 7525 4025 50  0000 L BNN
 F 1 "DS18B20" H 7525 3925 50  0000 L BNN
-F 2 "Housings_TO-92:TO-92_Molded_Narrow" H 7300 4150 50  0001 C CNN
+F 2 "onewire:1wire-TO92-" H 7300 4150 50  0001 C CNN
 F 3 "" H 7300 4000 60  0000 C CNN
 	3    7300 4000
@@
 Text Label 8450 2250 0    60   ~ 0
 tx
+$Comp
+L SW_PUSH SW1
+U 1 1 55A4108A
+P 3450 3900
+F 0 "SW1" H 3600 4010 50  0000 C CNN
+F 1 "SW_PUSH" H 3450 3820 50  0000 C CNN
+F 2 "Buttons_Switches_ThroughHole:SW_PUSH_SMALL" H 3450 3900 60  0001 C CNN
+F 3 "" H 3450 3900 60  0000 C CNN
+	1    3450 3900
+	1    0    0    -1
+$EndComp
 $EndSCHEMATC
