File: esp-humidity/esp-humidity.kicad_pcb (KiCad board)
At the start: 2 copper layers, 55.9 x 44.5 mm, 16 parts, among them Q1 IRLR3715ZPBF, U1 dht11, U2 esp8266-breakout

Commit message: fixed all the pcb mistakes
Parts:
- Q1: value IRLR3715ZPBF -> BUK98150-55A; footprint TO_SOT_Packages_SMD:TO-252-2Lead -> TO_SOT_Packages_SMD:SOT-223
- moved R3 12.7 mm to (143.5, 119.4), turned to 90 degrees
- moved Q1 4.32 mm to (151.6, 121.9)
Connections:
- Q1 pad 1: Net-(Q1-Pad1) -> /fan
- Q1 pad 2: /fan -> Net-(Q1-Pad2)
- U2 pad 10: Net-(U2-Pad10) -> /fan
- U2 pad 11: (no net) -> /gpio1
- U2 pad 12: (no net) -> /gpio2
- U2 pad 7: /fan -> (no net)
- U2 pad 9: Net-(U2-Pad9) -> (no net)
- fan1 pad 2: Net-(Q1-Pad1) -> Net-(Q1-Pad2)
- gpio1 pad 3: Net-(U2-Pad10) -> /gpio2
- gpio1 pad 4: Net-(U2-Pad9) -> /gpio1
Routing:
- net /gpio2: track 0.00 -> 27.4 mm
- net /gpio1: track 0.00 -> 25.2 mm
- net Net-(U2-Pad10): track 24.9 -> 0.00 mm
- net Net-(U2-Pad9): track 24.1 -> 0.00 mm
- net /fan: track 58.7 -> 74.9 mm, vias 0 -> 2
- net Net-(Q1-Pad1): track 8.83 -> 0.00 mm
- net Net-(Q1-Pad2): track 0.00 -> 8.64 mm
- net Earth: track 130.0 -> 126.6 mm
- net /status: track 22.5 -> 21.4 mm
- net /dht11-data: track 32.4 -> 31.7 mm
