File: modbox-lcd/modbox-lcd.kicad_pcb (KiCad board)
At the start: 2 copper layers, 100 x 40 mm, 24 parts, among them IC1 ATTINY88-A, P1 CONN_01X04, P2 CONN_02X03, P3 CONN_01X04, Q1 MMBF170, U1 tps61040

Commit message: new footprints, dc boost tested, ready for fab
Parts:
- added P4: CONN_01X04, Pin_Headers:Pin_Header_Straight_1x04, F.Cu at (210.5, 67.5)
- added REF**1: via, fp:via, F.Cu at (193.5, 78.5)
- added REF**10: via, fp:via, F.Cu at (189.5, 69.0)
- added REF**11: via, fp:via, F.Cu at (194.0, 73.5)
- added REF**12: via, fp:via, F.Cu at (195.0, 68.5)
- added REF**13: via, fp:via, F.Cu at (193.0, 63.5)
- added REF**14: via, fp:via, F.Cu at (192.0, 63.5)
- added REF**15: via, fp:via, F.Cu at (191.0, 63.5)
- added REF**2: via, fp:via, F.Cu at (192.5, 78.5)
- added REF**6: via, fp:via, F.Cu at (193.0, 73.5)
- added REF**7: via, fp:via, F.Cu at (188.5, 69.0)
- added REF**8: via, fp:via, F.Cu at (194.5, 78.5)
- added REF**9: via, fp:via, F.Cu at (191.5, 78.5)
- added SW1: SW_PUSH, fp:button, F.Cu at (210.4, 79.8)
- C5: value 1u -> 10u; footprint Capacitors_SMD:C_1206 -> SMD_Packages:SMD-1206_Pol
- C7: value 10u -> 1u
- L1: footprint Inductors_NEOSID:Neosid_Inductor_SMs50 -> Inductors_NEOSID:Neosid_Inductor_SMS-ME3015
- R1: value R -> 10k
- R5: value 620k -> 1m
- RV1: footprint SMD_Packages:POT_SMD -> fp:3mm pot
- moved R5 67.8 mm to (210.6, 72.2), turned to 0 degrees
- moved R1 22.4 mm to (148.5, 75.5), turned to 180 degrees
- moved RV1 2.00 mm to (119.0, 78.0), turned to 180 degrees
Connections:
- DS1 pad 15: Net-(DS1-Pad15) -> +5V
- IC1 pad 1: (no net) -> Net-(IC1-Pad1)
- IC1 pad 25: (no net) -> butt
- IC1 pad 30: (no net) -> Net-(IC1-Pad30)
- IC1 pad 31: (no net) -> Net-(IC1-Pad31)
- IC1 pad 32: (no net) -> Net-(IC1-Pad32)
- R1 pad 1: Net-(DS1-Pad15) -> pwm
- R1 pad 2: +5V -> Earth
- R5 pad 2: (no net) -> Net-(R5-Pad2)
Routing:
- net Net-(IC1-Pad30): track 0.00 -> 51.3 mm, vias 0 -> 1
- net Net-(IC1-Pad31): track 0.00 -> 51.2 mm, vias 0 -> 1
- net Net-(IC1-Pad32): track 0.00 -> 50.2 mm, vias 0 -> 1
- net Net-(IC1-Pad1): track 0.00 -> 49.6 mm, vias 0 -> 1
- net butt: track 0.00 -> 45.3 mm, vias 0 -> 2
- net Earth: track 101.9 -> 114.2 mm
- net Net-(DS1-Pad15): track 7.14 -> 0.00 mm
- net Net-(R5-Pad2): track 0.00 -> 6.87 mm
- net pwm: track 15.5 -> 19.8 mm
- net +5V: track 122.6 -> 125.9 mm
- net +3V3: track 152.7 -> 154.8 mm
- net Net-(DS1-Pad3): track 11.9 -> 12.8 mm, vias 2 -> 0
- net Net-(DS1-Pad16): track 46.1 -> 46.6 mm
Other:
- board text added: "0v 3.3v sda scl"
- board text added: "contrast"
- board text added: "gpio"

Commit message: tofab
Other:
- board text added: "lcd v0.1"
- board text removed: "encoder v0.1"
Changed lines of the file:
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@@
     (links 82)
     (no_connects 0)
-    (area 112.511474 39.14 219.490046 97.100001)
+    (area 114.949999 49.949999 215.050001 90.050001)
     (thickness 1.6)
     (drawings 52)
@@
     (effects (font (size 1.5 1.5) (thickness 0.3)))
   )
-  (gr_text "encoder v0.1" (at 130.1 87.8) (layer F.SilkS)
+  (gr_text "lcd v0.1" (at 130.1 87.8) (layer F.SilkS)
     (effects (font (size 1.5 1.5) (thickness 0.3)))
   )
