File: lucy-ren-badge/lucy-ren-badge.kicad_pcb (KiCad board)
At the start: 2 copper layers, 72.1 x 50.5 mm, 13 parts, among them J1 Conn_02x03_Odd_Even, SW1 SW_DIP_x01, U1 ATTINY88-AU, U2 rgbled

Commit message: commit before order
Parts:
- removed BT1: Battery_Cell, Battery_Holders:Keystone_3000_1x12mm-CoinCell
- added CR1220: Battery_Cell, fp:Keystone_3000_1x12mm-CoinCell, B.Cu at (145.8, 91.5)
- SW1: value SW_DIP_x01 -> SW_DIP_x02; footprint Buttons_Switches_SMD:SW_DIP_x1_W5.08mm_Slide_Copal_CHS-A -> raise_fp:SW_DIP_SPSTx02_Slide_6.7x6.64mm_W6.73mm_P2.54mm_LowProfile_JPin
- U2: footprint raise_fp:3528-4p -> fp:3528-4p
- moved R2 21.3 mm to (136.1, 82.6)
- moved R1 3.51 mm to (158.6, 79.0)
- moved J1 2.93 mm to (161.5, 69.5), turned to 180 degrees
- moved C1 2.79 mm to (158.6, 82.9), turned to 180 degrees
- moved SW1 2.13 mm to (125.1, 77.4)
- moved C2 1.77 mm to (133.6, 71.5)
- moved G*** 0.23 mm to (146.6, 81.3)
- moved G*** 0.22 mm to (146.6, 81.4)
- moved U2 0.13 mm to (143.7, 82.6)
Connections:
- SW1 pad 1: VCC -> /mode
- SW1 pad 2: Net-(BT1-Pad1) -> VCC
- U1 pad 19: Net-(U1-Pad19) -> /mode
Routing:
- net GND: track 0.00 -> 103.2 mm
- net VCC: track 0.00 -> 82.0 mm, vias 0 -> 7
- net /mode: track 0.00 -> 47.8 mm, vias 0 -> 4
- net Net-(BT1-Pad1): track 0.00 -> 36.1 mm
- net Net-(R2-Pad1): track 0.00 -> 33.8 mm, vias 0 -> 2
- net /reset: track 0.00 -> 23.1 mm
- net /b1: track 0.00 -> 21.7 mm, vias 0 -> 3
- net /g1: track 0.00 -> 21.2 mm, vias 0 -> 3
- net /mosi: track 0.00 -> 19.4 mm
- net /sck: track 0.00 -> 11.9 mm
- net /miso: track 0.00 -> 9.44 mm
- net /r1: track 0.00 -> 5.87 mm, vias 0 -> 1
Other:
- outline, holes or cut-outs redrawn
- net class Default: clearance 0.2 -> 0.16; trace_width 0.25 -> 0.16; via_dia 0.8 -> 0.6; via_drill 0.4 -> 0.3
- rule trace_clearance: 0.2 -> 0.16
- rule trace_min: 0.2 -> 0.16
- board text added: "mis sck rst"
- board text added: "mode"
- board text added: "mos gnd"
- board text added: "off"
- board text added: "on"
- board text added: "p1"

Commit message: track spacing
Routing:
- net GND: track 103.2 -> 104.7 mm
- net VCC: track 82.0 -> 82.7 mm
- net /g1: track 21.2 -> 21.8 mm
Other:
- board text added: "Matt Venn"

Commit message: add Rachel
Other:
- board text added: "Rachel Bollen"
